File: 281D.kicad_pcb (KiCad board)
At the start: 4 copper layers, 104 x 158 mm, 380 parts, among them J1 Q, J101 108-0906-001, J102 108-0903-001, J103 108-0903-001, J104 108-0902-001, J105 108-0910-001, J106 108-0910-001, J2 -15V, J201 108-0906-001, J202 108-0903-001, J203 108-0903-001, J204 108-0902-001, J205 108-0910-001, J3 +15V, J301 108-0906-001, J302 108-0903-001, J303 108-0903-001, J304 108-0902-001, J305 108-0910-001, J306 108-0910-001, J4 +12V, J401 108-0906-001, J402 108-0903-001, J403 108-0903-001, J404 108-0902-001, J405 108-0910-001, M1 Logo_150mil, M2 Mod_Indicator_1-10_150mil, M3 Serial_Box_150mil, Q1 MMBT3904, Q101 DMMT3906W, Q102 MMBFJ201, Q103 MMBT3904, Q201 DMMT3906W, Q202 MMBFJ201, Q203 MMBT3904, Q301 DMMT3906W, Q302 MMBFJ201, Q303 MMBT3904, Q401 DMMT3906W, Q402 MMBFJ201, Q403 MMBT3904, SW1 SPDT_ON-OFF-ON, SW101 SPDT_ON-OFF-ON, SW102 SPDT_ON-ON, SW201 SPDT_ON-OFF-ON, SW301 SPDT_ON-OFF-ON, SW302 SPDT_ON-ON, SW401 SPDT_ON-OFF-ON, U1 L78L10, U101 TL074, U102 4001, U103/203 4066, U104/204 LM13700, U105/205 TL074, U2 TL072, U201 TL074, U202 4001, U301 TL074, U302 4001, U303/403 4066, U304/404 LM13700, U305/405 TL074, U401 TL074, U402 4001

Commit message: Update BOM, BOM pdf, notes. Schematic and assembly guide correction.
Parts:
- C2: value 22uF -> 22u
- R2: value 20k -> 22k
Changed lines of the file:
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@@
-(kicad_pcb (version 20171130) (host pcbnew 5.1.5-1.fc30)
+(kicad_pcb (version 20171130) (host pcbnew 5.1.5-2.fc32)
   (general
     (thickness 1.6)
@@
       (effects (font (size 1 1) (thickness 0.15)) (justify mirror))
     )
-    (fp_text value 22uF (at 0 -3.7) (layer B.Fab)
+    (fp_text value 22u (at 0 -3.7) (layer B.Fab)
       (effects (font (size 1 1) (thickness 0.15)) (justify mirror))
     )
@@
       (effects (font (size 1 1) (thickness 0.15)) (justify mirror))
     )
-    (fp_text value 20k (at 0 -1.65 90) (layer B.Fab)
+    (fp_text value 22k (at 0 -1.65 90) (layer B.Fab)
       (effects (font (size 1 1) (thickness 0.15)) (justify mirror))
     )
