File: 281D.sch (KiCad schematic (older format))
At the start: 38 parts, among them J1 Q, J106 108-0910-001, J2 -15V, J3 +15V, J306 108-0910-001, J4 +12V, M1 Logo_150mil, M2 Mod_Indicator_1-10_150mil, M3 Serial_Box_150mil, Q1 MMBT3904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

Commit message: Update BOM, BOM pdf, notes. Schematic and assembly guide correction.
Parts:
- M1: symbol Dunnington:Logo_150mil -> 281D-rescue:Logo_150mil-Dunnington
- M2: symbol Dunnington:Mod_Indicator_1-10_150mil -> 281D-rescue:Mod_Indicator_1-10_150mil-Dunnington
- M3: symbol Dunnington:Serial_Box_150mil -> 281D-rescue:Serial_Box_150mil-Dunnington
- R2: value 20k -> 22k
Changed lines of the file:
@@
 P 3800 5000
 F 0 "R2" V 3725 5000 50  0000 C CNN
-F 1 "20k" V 3650 5000 50  0000 C CNN
+F 1 "22k" V 3650 5000 50  0000 C CNN
 F 2 "Resistor_SMD:R_0805_2012Metric" H 3800 5000 50  0001 C CNN
 F 3 "~" H 3800 5000 50  0001 C CNN
@@
 	3200 2700 3600 2700
 $Comp
-L Dunnington:Logo_150mil M1
+L 281D-rescue:Logo_150mil-Dunnington M1
 U 1 1 5E5809A9
 P 2450 6825
@@
 $EndComp
 $Comp
-L Dunnington:Mod_Indicator_1-10_150mil M2
+L 281D-rescue:Mod_Indicator_1-10_150mil-Dunnington M2
 U 1 1 5E58151D
 P 2450 7125
@@
 $EndComp
 $Comp
-L Dunnington:Serial_Box_150mil M3
+L 281D-rescue:Serial_Box_150mil-Dunnington M3
 U 1 1 5E5824E1
 P 2450 7400
